File: schematics/chip_counter.sch (EAGLE design)
At the start: 13 parts, among them U1 COMPUTE_MODULE

Commit message: update schematics
Connections:
- removed net N$2: RELAY-MOTOR1.5, RELAY-MOTOR2.5, TCRT5000-SENSOR_COUNT1.CATHODE, TCRT5000-SENSOR_COUNT2.CATHODE, TCRT5000-SENSOR_MOTOR1.CATHODE, TCRT5000-SENSOR_MOTOR2.CATHODE, U1.GND@57
- net MOTOR_GND: now also R1.3, R2.3
- net N$7: now also RELAY-MOTOR1.5, RELAY-MOTOR2.5, TCRT5000-SENSOR_COUNT1.CATHODE, TCRT5000-SENSOR_COUNT2.CATHODE, TCRT5000-SENSOR_MOTOR1.CATHODE, TCRT5000-SENSOR_MOTOR2.CATHODE, U1.GND@57; no longer U1.5V@1
Changed lines of the file:
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@@
-</segment>
-</net>
-<net name="N$2" class="0">
-<segment>
-<pinref part="TCRT5000-SENSOR_MOTOR1" gate="OS" pin="CATHODE"/>
-<pinref part="U1" gate="G$1" pin="GND@57"/>
-<wire x1="-91.44" y1="-73.66" x2="-91.44" y2="-119.38" width="0.1524" layer="91"/>
-<wire x1="-91.44" y1="-119.38" x2="-73.66" y2="-119.38" width="0.1524" layer="91"/>
-<pinref part="TCRT5000-SENSOR_MOTOR2" gate="OS" pin="CATHODE"/>
-<wire x1="-73.66" y1="-119.38" x2="-55.88" y2="-119.38" width="0.1524" layer="91"/>
-<wire x1="-55.88" y1="-119.38" x2="-35.56" y2="-119.38" width="0.1524" layer="91"/>
-<wire x1="-35.56" y1="-119.38" x2="-7.62" y2="-119.38" width="0.1524" layer="91"/>
-<wire x1="-73.66" y1="-73.66" x2="-73.66" y2="-119.38" width="0.1524" layer="91"/>
-<junction x="-73.66" y="-119.38"/>
-<pinref part="TCRT5000-SENSOR_COUNT1" gate="OS" pin="CATHODE"/>
-<wire x1="-55.88" y1="-73.66" x2="-55.88" y2="-119.38" width="0.1524" layer="91"/>
-<junction x="-55.88" y="-119.38"/>
-<pinref part="TCRT5000-SENSOR_COUNT2" gate="OS" pin="CATHODE"/>
-<wire x1="-35.56" y1="-73.66" x2="-35.56" y2="-119.38" width="0.1524" layer="91"/>
-<junction x="-35.56" y="-119.38"/>
-<pinref part="RELAY-MOTOR1" gate="G$1" pin="5"/>
-<wire x1="-91.44" y1="-119.38" x2="-106.68" y2="-119.38" width="0.1524" layer="91"/>
-<wire x1="-106.68" y1="-119.38" x2="-106.68" y2="-12.7" width="0.1524" layer="91"/>
-<junction x="-91.44" y="-119.38"/>
-<wire x1="-106.68" y1="-12.7" x2="-106.68" y2="0" width="0.1524" layer="91"/>
-<wire x1="-106.68" y1="-12.7" x2="-154.94" y2="-12.7" width="0.1524" layer="91"/>
-<pinref part="RELAY-MOTOR2" gate="G$1" pin="5"/>
-<wire x1="-154.94" y1="-12.7" x2="-154.94" y2="0" width="0.1524" layer="91"/>
 </segment>
 </net>
@@
 <pinref part="BUTTON-RESET" gate="1" pin="2"/>
 <wire x1="-22.86" y1="33.02" x2="-25.4" y2="33.02" width="0.1524" layer="91"/>
-<pinref part="U1" gate="G$1" pin="5V@1"/>
 <wire x1="-25.4" y1="33.02" x2="-25.4" y2="15.24" width="0.1524" layer="91"/>
-<wire x1="-25.4" y1="15.24" x2="-25.4" y2="-121.92" width="0.1524" layer="91"/>
-<wire x1="-25.4" y1="-121.92" x2="-7.62" y2="-121.92" width="0.1524" layer="91"/>
 <pinref part="BUTTON-MOTOR-ACTIVATION" gate="1" pin="2"/>
 <wire x1="-25.4" y1="33.02" x2="-25.4" y2="93.98" width="0.1524" layer="91"/>
@@
 <junction x="-25.4" y="33.02"/>
 <pinref part="KEYSWITCH" gate="G$1" pin="1"/>
+<pinref part="TCRT5000-SENSOR_MOTOR1" gate="OS" pin="CATHODE"/>
+<pinref part="U1" gate="G$1" pin="GND@57"/>
+<wire x1="-91.44" y1="-73.66" x2="-91.44" y2="-119.38" width="0.1524" layer="91"/>
+<wire x1="-91.44" y1="-119.38" x2="-73.66" y2="-119.38" width="0.1524" layer="91"/>
+<pinref part="TCRT5000-SENSOR_MOTOR2" gate="OS" pin="CATHODE"/>
+<wire x1="-73.66" y1="-119.38" x2="-55.88" y2="-119.38" width="0.1524" layer="91"/>
+<wire x1="-55.88" y1="-119.38" x2="-35.56" y2="-119.38" width="0.1524" layer="91"/>
+<wire x1="-35.56" y1="-119.38" x2="-25.4" y2="-119.38" width="0.1524" layer="91"/>
+<wire x1="-25.4" y1="-119.38" x2="-7.62" y2="-119.38" width="0.1524" layer="91"/>
+<wire x1="-73.66" y1="-73.66" x2="-73.66" y2="-119.38" width="0.1524" layer="91"/>
+<junction x="-73.66" y="-119.38"/>
+<pinref part="TCRT5000-SENSOR_COUNT1" gate="OS" pin="CATHODE"/>
+<wire x1="-55.88" y1="-73.66" x2="-55.88" y2="-119.38" width="0.1524" layer="91"/>
+<junction x="-55.88" y="-119.38"/>
+<pinref part="TCRT5000-SENSOR_COUNT2" gate="OS" pin="CATHODE"/>
+<wire x1="-35.56" y1="-73.66" x2="-35.56" y2="-119.38" width="0.1524" layer="91"/>
+<junction x="-35.56" y="-119.38"/>
+<pinref part="RELAY-MOTOR1" gate="G$1" pin="5"/>
+<wire x1="-91.44" y1="-119.38" x2="-106.68" y2="-119.38" width="0.1524" layer="91"/>
+<wire x1="-106.68" y1="-119.38" x2="-106.68" y2="-12.7" width="0.1524" layer="91"/>
+<junction x="-91.44" y="-119.38"/>
+<wire x1="-106.68" y1="-12.7" x2="-106.68" y2="0" width="0.1524" layer="91"/>
+<wire x1="-106.68" y1="-12.7" x2="-154.94" y2="-12.7" width="0.1524" layer="91"/>
+<pinref part="RELAY-MOTOR2" gate="G$1" pin="5"/>
+<wire x1="-154.94" y1="-12.7" x2="-154.94" y2="0" width="0.1524" layer="91"/>
+<wire x1="-25.4" y1="15.24" x2="-25.4" y2="-119.38" width="0.1524" layer="91"/>
 <junction x="-25.4" y="15.24"/>
+<junction x="-25.4" y="-119.38"/>
 </segment>
 </net>
@@
 <segment>
 <pinref part="SOURCE" gate="G$1" pin="-"/>
-<wire x1="-218.44" y1="53.34" x2="-218.44" y2="-60.96" width="0.1524" layer="91"/>
+<wire x1="-218.44" y1="53.34" x2="-218.44" y2="-40.64" width="0.1524" layer="91"/>
 <label x="-218.44" y="-60.96" size="1.778" layer="95"/>
+<pinref part="R2" gate="G$1" pin="3"/>
+<wire x1="-218.44" y1="-40.64" x2="-218.44" y2="-60.96" width="0.1524" layer="91"/>
+<wire x1="-185.42" y1="-40.64" x2="-218.44" y2="-40.64" width="0.1524" layer="91"/>
+<junction x="-218.44" y="-40.64"/>
+<pinref part="R1" gate="G$1" pin="3"/>
+<wire x1="-137.16" y1="-40.64" x2="-218.44" y2="-40.64" width="0.1524" layer="91"/>
 </segment>
 </net>
